Commit message: Start to implement a second intelligence with 2 cameras. Image acquisition already done.

File: p_vbatista/p_vbatista_description/urdf/p_vbatista.gazebo.macro.xacro (robot description, xacro)
@@ -144,4 +144,6 @@
         </gazebo>
       <!--link : https://www.raspberrypi.org/documentation/hardware/camera/-->
+        <!--Cameras-->
+              <!-- Camera Front -->
         <gazebo reference="camera_rgb_frame">
           <sensor type="camera" name="Pi Camera">
@@ -151,5 +153,5 @@
                 <horizontal_fov>1.085595</horizontal_fov>
                 <image>
-                    <width>640</width>
+                    <width>900</width>
                     <height>480</height>
                     <format>R8G8B8</format>
@@ -176,4 +178,37 @@
           </sensor>
         </gazebo>
+      <!-- Camera Back -->
+        <gazebo reference="camera_rgb_frame_2">
+          <sensor type="camera" name="Pi Camera 2">
+            <always_on>true</always_on>
+            <visualize>${camera_visual}</visualize>
+            <camera>
+                <horizontal_fov>1.085595</horizontal_fov>
+                <image>
+                    <width>900</width>
+                    <height>480</height>
+                    <format>R8G8B8</format>
+                </image>
+                <clip>
+                    <near>0.03</near>
+                    <far>100</far>
+                </clip>
+            </camera>
+            <plugin name="camera_controller" filename="libgazebo_ros_camera.so">
+              <alwaysOn>true</alwaysOn>
+              <updateRate>30.0</updateRate>
+              <cameraName>camera_2</cameraName>
+              <frameName>camera_rgb_optical_frame_2</frameName>
+              <imageTopicName>rgb/image_raw</imageTopicName>
+              <cameraInfoTopicName>camera_2/rgb/camera_info</cameraInfoTopicName>
+              <hackBaseline>0.07</hackBaseline>
+              <distortionK1>0.0</distortionK1>
+              <distortionK2>0.0</distortionK2>
+              <distortionK3>0.0</distortionK3>
+              <distortionT1>0.0</distortionT1>
+              <distortionT2>0.0</distortionT2>
+            </plugin>
+          </sensor>
+        </gazebo>
     </xacro:macro>
 </robot>

File: p_vbatista/p_vbatista_description/urdf/p_vbatista.urdf.xacro (robot description, xacro)
@@ -177,4 +177,5 @@
   </link>
 <!--  Cameras-->
+  <!-- Camera Front -->
   <joint name="camera_joint" type="fixed">
     <origin xyz="0.073 -0.011 0.084" rpy="0 0 0"/>
@@ -202,3 +203,29 @@
   </joint>
   <link name="camera_rgb_optical_frame"/>
+  <!-- Camera Back -->
+  <joint name="camera_joint_2" type="fixed">
+    <origin xyz="-0.2 -0.011 0.084" rpy="0 0 -3.14"/>
+    <parent link="base_link"/>
+    <child link="camera_link_2"/>
+  </joint>
+  <link name="camera_link_2">
+    <collision>
+      <origin xyz="0.005 0.011 0.013" rpy="0 0 0"/>
+      <geometry>
+        <box size="0.015 0.030 0.027"/>
+      </geometry>
+    </collision>
+  </link>
+  <joint name="camera_rgb_joint_2" type="fixed">
+    <origin xyz="0.003 0.011 0.009" rpy="0 0 0"/>
+    <parent link="camera_link_2"/>
+    <child link="camera_rgb_frame_2"/>
+  </joint>
+  <link name="camera_rgb_frame_2"/>
+  <joint name="camera_rgb_optical_joint_2" type="fixed">
+    <origin xyz="0 0 0" rpy="-1.57 0 -1.57"/>
+    <parent link="camera_rgb_frame_2"/>
+    <child link="camera_rgb_optical_frame_2"/>
+  </joint>
+  <link name="camera_rgb_optical_frame_2"/>
 </robot>
